File: WeatherStation.brd (EAGLE design)
At the start: 30.5 x 53.3 mm, 36 parts, among them J1 EDISON_CONNECTOR_FULLMOUNTING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, J2 EDISON_CONNECTOR_FULLHEADER, U1 MCP73831, U2 HTU21D, U3 MPL3115A2, U4 PCA9306

Commit message: corrected values
Parts:
- C11, C8: value 4.7µF -> 0.1µF
- C3, C4: value 4.7µF -> 2.2µF
- C5: value 4.7µF -> 470pF
- R2: value 330Ω -> 470Ω
- R5: value 1kΩ -> 200kΩ
Changed lines of the file:
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@@
 <attribute name="VALUE" x="9.5885" y="16.256" size="0.4064" layer="27" rot="R270"/>
 </element>
-<element name="R2" library="SparkFun-Resistors" package="0603-RES" value="330Ω" x="10.668" y="12.192" smashed="yes" rot="R90">
+<element name="R2" library="SparkFun-Resistors" package="0603-RES" value="470Ω" x="10.668" y="12.192" smashed="yes" rot="R90">
 <attribute name="VALUE" x="9.779" y="12.192" size="0.4064" layer="27" rot="R90" align="center"/>
 </element>
@@
 <attribute name="VALUE" x="7.3025" y="24.1935" size="0.4064" layer="27" rot="R90" align="center"/>
 </element>
-<element name="C3" library="SparkFun-Capacitors" package="0805" value="4.7µF" x="7.366" y="21.59" smashed="yes">
+<element name="C3" library="SparkFun-Capacitors" package="0805" value="2.2µF" x="7.366" y="21.59" smashed="yes">
 <attribute name="VALUE" x="8.89" y="21.463" size="0.4064" layer="27"/>
 </element>
-<element name="C4" library="SparkFun-Capacitors" package="0805" value="4.7µF" x="7.366" y="26.67" smashed="yes" rot="R180">
+<element name="C4" library="SparkFun-Capacitors" package="0805" value="2.2µF" x="7.366" y="26.67" smashed="yes" rot="R180">
 <attribute name="VALUE" x="8.382" y="28.067" size="0.4064" layer="27" rot="R180"/>
 </element>
-<element name="C5" library="SparkFun-Capacitors" package="0805" value="4.7µF" x="10.922" y="24.13" smashed="yes" rot="R90">
+<element name="C5" library="SparkFun-Capacitors" package="0805" value="470pF" x="10.922" y="24.13" smashed="yes" rot="R90">
 <attribute name="VALUE" x="11.811" y="24.13" size="0.4064" layer="27" rot="R90" align="top-center"/>
 </element>
@@
 <attribute name="VALUE" x="5.842" y="34.671" size="0.4064" layer="27"/>
 </element>
-<element name="R5" library="SparkFun-Resistors" package="0603-RES" value="1kΩ" x="14.224" y="30.48" smashed="yes">
+<element name="R5" library="SparkFun-Resistors" package="0603-RES" value="200kΩ" x="14.224" y="30.48" smashed="yes">
 <attribute name="VALUE" x="11.684" y="30.353" size="0.4064" layer="27"/>
 </element>
@@
 <attribute name="VALUE" x="11.684" y="26.289" size="0.4064" layer="27"/>
 </element>
-<element name="C8" library="SparkFun-Capacitors" package="0805" value="4.7µF" x="7.112" y="51.816" smashed="yes">
+<element name="C8" library="SparkFun-Capacitors" package="0805" value="0.1µF" x="7.112" y="51.816" smashed="yes">
 <attribute name="VALUE" x="7.112" y="50.927" size="0.4064" layer="27" align="top-center"/>
 </element>
@@
 <attribute name="VALUE" x="26.478" y="48.106" size="0.4064" layer="27" rot="R270"/>
 </element>
-<element name="C11" library="SparkFun-Capacitors" package="0805" value="4.7µF" x="13.716" y="33.782" smashed="yes" rot="R90">
+<element name="C11" library="SparkFun-Capacitors" package="0805" value="0.1µF" x="13.716" y="33.782" smashed="yes" rot="R90">
 <attribute name="VALUE" x="15.113" y="32.766" size="0.4064" layer="27" rot="R90"/>
 </element>
